Commit message: continuous

File: src/puck_description/xacro/puck_base.xacro (robot description, xacro)
@@ -30,5 +30,5 @@
             </visual>
         </link>
-		<joint name="base_to_${prefix}_wheel" type="fixed">
+		<joint name="base_to_${prefix}_wheel" type="continuous">
             <parent link="base_link"/>
             <child link="${prefix}_wheel"/>
